File: pcb/motor-driver.kicad_sch (KiCad schematic)
At the start: 14 parts, among them J3 B6B-PH-SM4-TB, U7 TMC2130-LA

Commit message: Add 3d parts
Parts:
- J3: footprint Connector_JST:JST_PH_B6B-PH-SM4-TB_1x06-1MP_P2.00mm_Vertical -> open-ephys:JST_PH_B6B-PH-SM4-TB_1x06-1MP_P2.00mm_Vertical
Changed lines of the file:
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@@
 			)
 		)
-		(property "Footprint" "Connector_JST:JST_PH_B6B-PH-SM4-TB_1x06-1MP_P2.00mm_Vertical"
+		(property "Footprint" "open-ephys:JST_PH_B6B-PH-SM4-TB_1x06-1MP_P2.00mm_Vertical"
 			(at 210.82 85.09 0)
 			(effects
