File: pcb/motor-driver.kicad_sch (KiCad schematic)
At the start: 15 parts, among them J3 1719730004, U7 TMC2130-LA

Commit message: Revision E
- Resolve issues 1-11
- Add pdf of rev d schematic for easy comparison
Parts:
- removed TP4: ~, TestPoint:TestPoint_Pad_D2.0mm, symbol Connector:TestPoint
- C27, C28, C31, C32: footprint Capacitor_SMD:C_0603_1608Metric -> Capacitor_SMD:C_0402_1005Metric
Connections:
- net +15V renamed +12V
Changed lines of the file:
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@@
-	)
-	(junction
-		(at 116.84 41.91)
-		(diameter 0)
-		(color 0 0 0 0)
 	)
 	(junction
@@
 			)
 		)
-		(property "Footprint" "Capacitor_SMD:C_0603_1608Metric"
+		(property "Footprint" "Capacitor_SMD:C_0402_1005Metric"
 			(at 117.8052 53.34 0)
 			(effects
@@
 	)
 	(symbol
-		(lib_id "Connector:TestPoint")
-		(at 116.84 41.91 0)
-		(unit 1)
-		(exclude_from_sim no)
-		(in_bom yes)
-		(on_board yes)
-		(dnp no)
-		(fields_autoplaced yes)
-		(property "Reference" "TP4"
-			(at 119.38 39.243 0)
-			(effects
-				(font
-					(size 1.27 1.27)
-				)
-				(justify left)
-			)
-		)
-		(property "Value" "~"
-			(at 119.38 40.513 0)
-			(effects
-				(font
-					(size 1.27 1.27)
-				)
-				(justify left)
-			)
-		)
-		(property "Footprint" "TestPoint:TestPoint_Pad_D2.0mm"
-			(at 121.92 41.91 0)
-			(effects
-				(font
-					(size 1.27 1.27)
-				)
-				(hide yes)
-			)
-		)
-		(property "Datasheet" "~"
-			(at 121.92 41.91 0)
-			(effects
-				(font
-					(size 1.27 1.27)
-				)
-				(hide yes)
-			)
-		)
-		(property "Description" "test point"
-			(at 116.84 41.91 0)
-			(effects
-				(font
-					(size 1.27 1.27)
-				)
-				(hide yes)
-			)
-		)
-		(pin "1"
-		)
-		(instances
-			(project "oe-commutator-controller"
-				(path "/f8e1d654-dc44-4fb2-953c-f5982945ff40/8643cb4c-0280-4c6b-b319-4ef16f8d0a00"
-					(reference "TP4")
-					(unit 1)
-				)
-			)
-		)
-	)
-	(symbol
 		(lib_id "power:+15V")
 		(at 186.69 39.37 0)
@@
 			)
 		)
-		(property "Value" "+15V"
+		(property "Value" "+12V"
 			(at 186.69 34.29 0)
 			(effects
@@
 			)
 		)
-		(property "Value" "+15V"
+		(property "Value" "+12V"
 			(at 176.53 34.29 0)
 			(effects
@@
 			)
 		)
-		(property "Footprint" "Capacitor_SMD:C_0603_1608Metric"
+		(property "Footprint" "Capacitor_SMD:C_0402_1005Metric"
 			(at 103.1748 45.72 0)
 			(effects
@@
 			)
 		)
-		(property "Footprint" "Capacitor_SMD:C_0603_1608Metric"
+		(property "Footprint" "Capacitor_SMD:C_0402_1005Metric"
 			(at 180.0352 63.5 0)
 			(effects
@@
 			)
 		)
-		(property "Value" "+15V"
+		(property "Value" "+12V"
 			(at 104.14 34.29 0)
 			(effects
@@
 			)
 		)
-		(property "Footprint" "Capacitor_SMD:C_0603_1608Metric"
+		(property "Footprint" "Capacitor_SMD:C_0402_1005Metric"
 			(at 175.5648 45.72 0)
 			(effects

Commit message: Revision F Edits
- Reduce base capacitance
  - Reduce infill {width, gap}: {0.35, 1} -> {0.2, 1.2}
    - Equivalent to: 45.1% -> 26.5%
  - Entirely remove copper on 3rd (in2.Cu) layer
  - Reduce via count
- export rev e schematic to pdf
- put pdfs into manufacturing folder
- Fix 6mm tactile switch footprint
- Put gold under logo
- Increment schematic, pcb, and silkscreen revision to F
- Add labels to debug header
- Add 10k pull-up to tmc2130 enable pin
- Convert all symbols & footprints library aliases from "oe" to "open-ephys"
Parts:
- added R31: 10k, Resistor_SMD:R_0603_1608Metric, symbol Device:R_US
- J3: footprint oe:MOLEX_1719730004_1x04_P2.54mm_Vert_Lock -> open-ephys:MOLEX_1719730004_1x04_P2.54mm_Vert_Lock
Connections:
- net +3.3V: now also R31.1
- net TMC_{EN}: now also R31.2
Changed lines of the file:
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@@
 	)
 	(junction
+		(at 101.6 113.03)
+		(diameter 0)
+		(color 0 0 0 0)
+	)
+	(junction
 		(at 176.53 44.45)
 		(diameter 0)
@@
 	(wire
 		(pts
+			(xy 101.6 111.76) (xy 101.6 113.03)
+		)
+		(stroke
+			(width 0)
+			(type default)
+		)
+	)
+	(wire
+		(pts
 			(xy 114.3 77.47) (xy 130.81 77.47)
 		)
@@
 	(wire
 		(pts
+			(xy 101.6 102.87) (xy 101.6 104.14)
+		)
+		(stroke
+			(width 0)
+			(type default)
+		)
+	)
+	(wire
+		(pts
 			(xy 162.56 44.45) (xy 162.56 45.72)
 		)
@@
 	(wire
 		(pts
+			(xy 101.6 113.03) (xy 130.81 113.03)
+		)
+		(stroke
+			(width 0)
+			(type default)
+		)
+	)
+	(wire
+		(pts
 			(xy 186.69 39.37) (xy 186.69 62.23)
 		)
@@
 	(wire
 		(pts
-			(xy 129.54 113.03) (xy 130.81 113.03)
+			(xy 97.79 113.03) (xy 101.6 113.03)
 		)
 		(stroke
@@
 	(hierarchical_label "TMC_{EN}"
 		(shape input)
-		(at 129.54 113.03 180)
+		(at 97.79 113.03 180)
 		(fields_autoplaced yes)
 		(effects
@@
 			)
 		)
-		(property "Footprint" "oe:MOLEX_1719730004_1x04_P2.54mm_Vert_Lock"
+		(property "Footprint" "open-ephys:MOLEX_1719730004_1x04_P2.54mm_Vert_Lock"
 			(at 176.53 96.52 0)
 			(effects
@@
 	)
 	(symbol
+		(lib_id "power:+3.3V")
+		(at 101.6 102.87 0)
+		(unit 1)
+		(exclude_from_sim no)
+		(in_bom yes)
+		(on_board yes)
+		(dnp no)
+		(fields_autoplaced yes)
+		(property "Reference" "#PWR038"
+			(at 101.6 106.68 0)
+			(effects
+				(font
+					(size 1.27 1.27)
+				)
+				(hide yes)
+			)
+		)
+		(property "Value" "+3.3V"
+			(at 101.6 97.79 0)
+			(effects
+				(font
+					(size 1.27 1.27)
+				)
+			)
+		)
+		(property "Footprint" ""
+			(at 101.6 102.87 0)
+			(effects
+				(font
+					(size 1.27 1.27)
+				)
+				(hide yes)
+			)
+		)
+		(property "Datasheet" ""
+			(at 101.6 102.87 0)
+			(effects
+				(font
+					(size 1.27 1.27)
+				)
+				(hide yes)
+			)
+		)
+		(property "Description" "Power symbol creates a global label with name \"+3.3V\""
+			(at 101.6 102.87 0)
+			(effects
+				(font
+					(size 1.27 1.27)
+				)
+				(hide yes)
+			)
+		)
+		(pin "1"
+		)
+		(instances
+			(project "oe-commutator-controller"
+				(path "/f8e1d654-dc44-4fb2-953c-f5982945ff40/8643cb4c-0280-4c6b-b319-4ef16f8d0a00"
+					(reference "#PWR038")
+					(unit 1)
+				)
+			)
+		)
+	)
+	(symbol
 		(lib_id "power:GND")
 		(at 176.53 54.61 0)
@@
 					(unit 1)
 				)
+			)
+		)
+	)
+	(symbol
+		(lib_id "Device:R_US")
+		(at 101.6 107.95 0)
+		(unit 1)
+		(exclude_from_sim no)
+		(in_bom yes)
+		(on_board yes)
+		(dnp no)
+		(fields_autoplaced yes)
+		(property "Reference" "R31"
+			(at 104.14 106.6799 0)
+			(effects
+				(font
+					(size 1.27 1.27)
+				)
+				(justify left)
+			)
+		)
+		(property "Value" "10k"
+			(at 104.14 109.2199 0)
+			(effects
+				(font
+					(size 1.27 1.27)
+				)
+				(justify left)
+			)
+		)
+		(property "Footprint" "Resistor_SMD:R_0603_1608Metric"
+			(at 102.616 108.204 90)
+			(effects
+				(font
+					(size 1.27 1.27)
+				)
+				(hide yes)
+			)
+		)
+		(property "Datasheet" "~"
+			(at 101.6 107.95 0)
+			(effects
+				(font
+					(size 1.27 1.27)
+				)
+				(hide yes)
+			)
+		)
+		(property "Description" "Resistor, US symbol"
+			(at 101.6 107.95 0)
+			(effects
+				(font
+					(size 1.27 1.27)
+				)
+				(hide yes)
+			)
+		)
+		(pin "2"
+		)
+		(pin "1"
+		)
+		(instances
+			(project ""
+				(path "/f8e1d654-dc44-4fb2-953c-f5982945ff40/8643cb4c-0280-4c6b-b319-4ef16f8d0a00"
+					(reference "R31")
+					(unit 1)
+				)

Commit message: Some edits during PR review
- Silkscreen moved on board
- Get rid of value text in fab layer
- Invert TMC_EN name to indicate correct logic
Connections:
- net TMC_{EN} renamed TMC_{~{EN}}
Changed lines of the file:
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@@
 		)
 	)
-	(hierarchical_label "TMC_{EN}"
+	(hierarchical_label "TMC_{~{EN}}"
 		(shape input)
 		(at 97.79 113.03 180)

Commit message: Address PCB issues found during testing
- Switch motor connector to JST PH
- Remove AIN_REF connection on TMC2130
- Replace sense resistors with 0.5 Ohm
Parts:
- removed R22: 30k, Resistor_SMD:R_0603_1608Metric, symbol Device:R_US
- J3: value 1719730004 -> B6B-PH-SM4-TB; footprint open-ephys:MOLEX_1719730004_1x04_P2.54mm_Vert_Lock -> Connector_JST:JST_PH_B6B-PH-SM4-TB_1x06-1MP_P2.00mm_Vertical; symbol Connector_Generic:Conn_01x04 -> Connector_Generic:Conn_01x06
- R20, R21: value 0.11,0.5W -> 0.5,0.5W; Tolerance (none) -> 1%
Connections:
- net OA1: now also J3.6 (Pin_6); no longer J3.2 (Pin_2)
- net OA2: now also J3.4 (Pin_4); no longer J3.1 (Pin_1)
- net OB2: now also J3.1 (Pin_1); no longer J3.4 (Pin_4)
- no-connect marks 4 -> 7
Other:
- note added: "NB: ~0.44A max I_{RMS} (pg. 55)"
- note removed: "NB: ~1.8A I_{peak} (pg. 55)"

Commit message: Add USB diode protection (#35)
- Change revision g -> h
  - schematic
  - pcb
  - silk screen
* Add 3d parts
Parts:
- J3: footprint Connector_JST:JST_PH_B6B-PH-SM4-TB_1x06-1MP_P2.00mm_Vertical -> open-ephys:JST_PH_B6B-PH-SM4-TB_1x06-1MP_P2.00mm_Vertical
Changed lines of the file:
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@@
 (kicad_sch
-	(version 20241209)
+	(version 20250114)
 	(generator "eeschema")
 	(generator_version "9.0")
@@
 			)
 		)
-		(property "Footprint" "Connector_JST:JST_PH_B6B-PH-SM4-TB_1x06-1MP_P2.00mm_Vertical"
+		(property "Footprint" "open-ephys:JST_PH_B6B-PH-SM4-TB_1x06-1MP_P2.00mm_Vertical"
 			(at 210.82 85.09 0)
 			(effects

Commit message: Lower sense resistance (0.5 -> 0.43 Ohms)
Also:
- Route TMC2130 diagnostic pins to RP2040
- Instead of manually excluding violations:
  - Changed spoke minimum: 2 -> 1
  - Changed copper-to-hole clearance: 0.25mm -> 0.19mm
- Update revision labels on sch, pcb, and silkscreen
Parts:
- R20, R21: value 0.5,0.5W -> 0.43,0.5W
Connections:
- net TMC_{DIAG0}: now reaches U7.20 (DIAG0)
- net TMC_{DIAG1}: now reaches U7.21 (DIAG1)
- no-connect marks 7 -> 5
Other:
- note removed: "NB: ~0.44A max I_{RMS} (pg. 55)"
Changed lines of the file:
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@@
 		(comment 2 "Jonathan P. Newman")
-	)
-	(text "NB: ~0.44A max I_{RMS}\n(pg. 55)"
-		(exclude_from_sim no)
-		(at 167.64 113.03 0)
-		(effects
-			(font
-				(size 1.27 1.27)
-			)
-			(justify left bottom)
-		)
 	)
 	(text "NB: Connect\nto GNDA"
@@
 	)
 	(no_connect
-		(at 130.81 118.11)
-	)
-	(no_connect
-		(at 130.81 120.65)
-	)
-	(no_connect
 		(at 130.81 102.87)
 	)
@@
 	(wire
 		(pts
+			(xy 125.73 118.11) (xy 130.81 118.11)
+		)
+		(stroke
+			(width 0)
+			(type default)
+		)
+	)
+	(wire
+		(pts
 			(xy 114.3 105.41) (xy 114.3 107.95)
 		)
@@
 		(pts
 			(xy 104.14 85.09) (xy 113.03 85.09)
+		)
+		(stroke
+			(width 0)
+			(type default)
+		)
+	)
+	(wire
+		(pts
+			(xy 125.73 120.65) (xy 130.81 120.65)
 		)
 		(stroke
@@
 			)
 			(justify left bottom)
+		)
+	)
+	(hierarchical_label "TMC_{DIAG1}"
+		(shape output)
+		(at 125.73 120.65 180)
+		(effects
+			(font
+				(size 1.27 1.27)
+			)
+			(justify right)
 		)
 	)
@@
 		(shape input)
 		(at 129.54 97.79 180)
+		(effects
+			(font
+				(size 1.27 1.27)
+			)
+			(justify right)
+		)
+	)
+	(hierarchical_label "TMC_{DIAG0}"
+		(shape output)
+		(at 125.73 118.11 180)
 		(effects
 			(font
@@
 			)
 		)
-		(property "Value" "0.5,0.5W"
+		(property "Value" "0.43,0.5W"
 			(at 182.88 124.46 0)
 			(effects
@@
 			)
 		)
-		(property "Value" "0.5,0.5W"
+		(property "Value" "0.43,0.5W"
 			(at 168.91 124.46 0)
 			(effects
