File: pcb/motor-driver.kicad_sch (KiCad schematic)
At the start: 14 parts, among them J3 B6B-PH-SM4-TB, U7 TMC2130-LA

Commit message: Complete OEPS PN and manufacturing files
Parts:
- C27, C28, C31, C32: MPN (none) -> CGA2B3X7R1H104K050BB; OEPS PN (none) -> OEPS010016
- C29: MPN (none) -> CL21B474KBFNNNG; OEPS PN (none) -> OEPS010099
- C30, C33: MPN (none) -> GRM21BR61H475KE51L; OEPS PN (none) -> OEPS010013
- C34: MPN (none) -> C1608X7R2A223K080AA; OEPS PN (none) -> OEPS010056
- J3: MPN (none) -> B6B-PH-SM4-TB; OEPS PN (none) -> OEPS070154
- R19: MPN (none) -> CRCW06032R20FKEAC; OEPS PN (none) -> OEPS020240
- R20, R21: MPN (none) -> KDV12DR470ET; OEPS PN (none) -> OEPS020241
- R31: MPN (none) -> RC0603FR-0710KL; OEPS PN (none) -> OEPS020133
- U7: MPN (none) -> TMC2130-LA; OEPS PN (none) -> OEPS080231
Changed lines of the file:
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@@
 			)
 		)
-		(property "Description" "Unpolarized capacitor"
+		(property "Description" "CAPACITOR:   SMD CER 0805 4.7uF 50V ±10% X5R   [GRM21BR61H475KE51L] [SMD]"
 			(at 186.69 67.31 0)
 			(hide yes)
@@
 			)
 		)
-		(property "MPN" ""
+		(property "MPN" "GRM21BR61H475KE51L"
 			(at 186.69 67.31 0)
 			(hide yes)
@@
 			)
 		)
-		(property "OEPS PN" ""
+		(property "OEPS PN" "OEPS010013"
 			(at 186.69 67.31 0)
 			(hide yes)
@@
 			)
 		)
-		(property "Description" "Resistor, US symbol"
+		(property "Description" "RESISTOR:   SMD 1206 0.47Ω ±0.5% 0.500W   [KDV12DR470ET] [SMD]"
 			(at 181.61 123.19 0)
 			(hide yes)
@@
 			)
 		)
-		(property "MPN" ""
+		(property "MPN" "KDV12DR470ET"
 			(at 181.61 123.19 0)
 			(hide yes)
@@
 			)
 		)
-		(property "OEPS PN" ""
+		(property "OEPS PN" "OEPS020241"
 			(at 181.61 123.19 0)
 			(hide yes)
@@
 			)
 		)
-		(property "Description" "Unpolarized capacitor"
+		(property "Description" "CAPACITOR:   SMD CER 0402 100nF 50V ±10% X7R   [CGA2B3X7R1H104K050BB] [SMD]"
 			(at 116.84 49.53 0)
 			(hide yes)
@@
 			)
 		)
-		(property "MPN" ""
+		(property "MPN" "CGA2B3X7R1H104K050BB"
 			(at 116.84 49.53 0)
 			(hide yes)
@@
 			)
 		)
-		(property "OEPS PN" ""
+		(property "OEPS PN" "OEPS010016"
 			(at 116.84 49.53 0)
 			(hide yes)
@@
 			)
 		)
-		(property "Description" "Resistor, US symbol"
+		(property "Description" "RESISTOR:   SMD 1206 0.47Ω ±0.5% 0.500W   [KDV12DR470ET] [SMD]"
 			(at 167.64 123.19 0)
 			(hide yes)
@@
 			)
 		)
-		(property "MPN" ""
+		(property "MPN" "KDV12DR470ET"
 			(at 167.64 123.19 0)
 			(hide yes)
@@
 			)
 		)
-		(property "OEPS PN" ""
+		(property "OEPS PN" "OEPS020241"
 			(at 167.64 123.19 0)
 			(hide yes)
@@
 			)
 		)
-		(property "Description" "Generic connector, single row, 01x06, script generated (kicad-library-utils/schlib/autogen/connector/)"
+		(property "Description" "CONNECTOR:   HEADER SMD JST 6POS 2MM   [B6B-PH-SM4-TB] [SMD]"
 			(at 210.82 85.09 0)
 			(hide yes)
@@
 			)
 		)
-		(property "MPN" ""
+		(property "MPN" "B6B-PH-SM4-TB"
 			(at 210.82 85.09 0)
 			(hide yes)
@@
 			)
 		)
-		(property "OEPS PN" ""
+		(property "OEPS PN" "OEPS070154"
 			(at 210.82 85.09 0)
 			(hide yes)
@@
 			)
 		)
-		(property "Description" "Unpolarized capacitor"
+		(property "Description" "CAPACITOR:   SMD CER 0603 22nF 100V ±10% X7R   [C1608X7R2A223K080AA] [SMD]"
 			(at 104.14 78.74 0)
 			(hide yes)
@@
 			)
 		)
-		(property "MPN" ""
+		(property "MPN" "C1608X7R2A223K080AA"
 			(at 104.14 78.74 0)
 			(hide yes)
@@
 			)
 		)
-		(property "OEPS PN" ""
+		(property "OEPS PN" "OEPS010056"
 			(at 104.14 78.74 0)
 			(hide yes)
@@
 			)
 		)
-		(property "Description" "Resistor, US symbol"
+		(property "Description" "RESISTOR:   SMD 0603 2.2Ω ±1% 0.100W   [CRCW06032R20FKEAC] [SMD]"
 			(at 152.4 44.45 0)
 			(hide yes)
@@
 			)
 		)
-		(property "MPN" ""
+		(property "MPN" "CRCW06032R20FKEAC"
 			(at 152.4 44.45 0)
 			(hide yes)
@@
 			)
 		)
-		(property "OEPS PN" ""
+		(property "OEPS PN" "OEPS020240"
 			(at 152.4 44.45 0)
 			(hide yes)
@@
 			)
 		)
-		(property "Description" "Unpolarized capacitor"
+		(property "Description" "CAPACITOR:   SMD CER 0805 470nF 50V ±10% X7R   [CL21B474KBFNNNG] [SMD]"
 			(at 129.54 49.53 0)
 			(hide yes)
@@
 			)
 		)
-		(property "MPN" ""
+		(property "MPN" "CL21B474KBFNNNG"
 			(at 129.54 49.53 0)
 			(hide yes)
@@
 			)
 		)
-		(property "OEPS PN" ""
+		(property "OEPS PN" "OEPS010099"
 			(at 129.54 49.53 0)
 			(hide yes)
@@
 			)
 		)
-		(property "Description" "Unpolarized capacitor"
+		(property "Description" "CAPACITOR:   SMD CER 0805 4.7uF 50V ±10% X5R   [GRM21BR61H475KE51L] [SMD]"
 			(at 162.56 49.53 0)
 			(hide yes)
@@
 			)
 		)
-		(property "MPN" ""
+		(property "MPN" "GRM21BR61H475KE51L"
 			(at 162.56 49.53 0)
 			(hide yes)
@@
 			)
 		)
-		(property "OEPS PN" ""
+		(property "OEPS PN" "OEPS010013"
 			(at 162.56 49.53 0)
 			(hide yes)
@@
 			)
 		)
-		(property "Description" "Unpolarized capacitor"
+		(property "Description" "CAPACITOR:   SMD CER 0402 100nF 50V ±10% X7R   [CGA2B3X7R1H104K050BB] [SMD]"
 			(at 104.14 49.53 0)
 			(hide yes)
@@
 			)
 		)
-		(property "MPN" ""
+		(property "MPN" "CGA2B3X7R1H104K050BB"
 			(at 104.14 49.53 0)
 			(hide yes)
@@
 			)
 		)
-		(property "OEPS PN" ""
+		(property "OEPS PN" "OEPS010016"
 			(at 104.14 49.53 0)
 			(hide yes)
@@
 			)
 		)
-		(property "Description" "Unpolarized capacitor"
+		(property "Description" "CAPACITOR:   SMD CER 0402 100nF 50V ±10% X7R   [CGA2B3X7R1H104K050BB] [SMD]"
 			(at 179.07 67.31 0)
 			(hide yes)
@@
 			)
 		)
-		(property "MPN" ""
+		(property "MPN" "CGA2B3X7R1H104K050BB"
 			(at 179.07 67.31 0)
 			(hide yes)
@@
 			)
 		)
-		(property "OEPS PN" ""
+		(property "OEPS PN" "OEPS010016"
 			(at 179.07 67.31 0)
 			(hide yes)
@@
 			)
 		)
-		(property "Description" "Driver for two-phase bipolar stepper motor, 2.0A, SPI, 4.75-46V, QFN-36"
+		(property "Description" "IC:   STEPPER MOTOR DRIVER   [TMC2130-LA] [36-QFN ]"
 			(at 148.59 102.87 0)
 			(hide yes)
@@
 			)
 		)
-		(property "MPN" ""
+		(property "MPN" "TMC2130-LA"
 			(at 148.59 102.87 0)
 			(hide yes)
@@
 			)
 		)
-		(property "OEPS PN" ""
+		(property "OEPS PN" "OEPS080231"
 			(at 148.59 102.87 0)
 			(hide yes)
@@
 			)
 		)
-		(property "Description" "Resistor, US symbol"
+		(property "Description" "RESISTOR:   SMD 0603 10kΩ ±1% 0.100W   [RC0603FR-0710KL] [SMD]"
 			(at 101.6 107.95 0)
 			(hide yes)
@@
 			)
 		)
-		(property "MPN" ""
+		(property "MPN" "RC0603FR-0710KL"
 			(at 101.6 107.95 0)
 			(hide yes)
@@
 			)
 		)
-		(property "OEPS PN" ""
+		(property "OEPS PN" "OEPS020133"
 			(at 101.6 107.95 0)
 			(hide yes)
@@
 			)
 		)
-		(property "Description" "Unpolarized capacitor"
+		(property "Description" "CAPACITOR:   SMD CER 0402 100nF 50V ±10% X7R   [CGA2B3X7R1H104K050BB] [SMD]"
 			(at 176.53 49.53 0)
 			(hide yes)
@@
 			)
 		)
-		(property "MPN" ""
+		(property "MPN" "CGA2B3X7R1H104K050BB"
 			(at 176.53 49.53 0)
 			(hide yes)
@@
 			)
 		)
-		(property "OEPS PN" ""
+		(property "OEPS PN" "OEPS010016"
 			(at 176.53 49.53 0)
 			(hide yes)
