File: pcb/cap-touch-sensor.kicad_sch (KiCad schematic)
At the start: 12 parts, among them U4 CAP1296-x-AIA

Commit message: Exclude test points and capacitive touch from assembly position files
Also raised KiCAD version from 9 to 10.

These are non-assembly components that should not be included in pick-and-place machine files.

If possible, the Attributes for Test Points and Mounting Holes should be:
[X]  Exclude from bill of materials
[  ]  Exclude from board
[X]  Exclude from position files
[  ]  Do not populate
Parts:
- S1, S2, S3, S4: value ~ -> (none)

Commit message: Complete OEPS PN and manufacturing files
Parts:
- C16: MPN (none) -> CL10A105KA8NNNC; OEPS PN (none) -> OEPS010022
- C19: MPN (none) -> C1005X5R1V104K050BB; OEPS PN (none) -> OEPS010066
- R25: MPN (none) -> RC0603FR-0710KL; OEPS PN (none) -> OEPS020133
- R32, R33, R34, R35: MPN (none) -> RC0805JR-070RL; OEPS PN (none) -> OEPS020025
- U4: MPN (none) -> CAP1296-1-AIA-TR; OEPS PN (none) -> OEPS080233
Changed lines of the file:
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@@
 			)
 		)
-		(property "Description" "Resistor, US symbol"
+		(property "Description" "RESISTOR:   SMD 0603 10kΩ ±1% 0.100W   [RC0603FR-0710KL] [SMD]"
 			(at 180.34 96.52 0)
 			(hide yes)
@@
 			)
 		)
-		(property "MPN" ""
+		(property "MPN" "RC0603FR-0710KL"
 			(at 180.34 96.52 0)
 			(hide yes)
@@
 			)
 		)
-		(property "OEPS PN" ""
+		(property "OEPS PN" "OEPS020133"
 			(at 180.34 96.52 0)
 			(hide yes)
@@
 			)
 		)
-		(property "Description" "Unpolarized capacitor"
+		(property "Description" "CAPACITOR:   SMD CER 0402 100nF 35V ±10% X5R (OEPS H1 001)   [C1005X5R1V104K050BB] [SMD]"
 			(at 147.32 80.01 0)
 			(hide yes)
@@
 			)
 		)
-		(property "MPN" ""
+		(property "MPN" "C1005X5R1V104K050BB"
 			(at 147.32 80.01 0)
 			(hide yes)
@@
 			)
 		)
-		(property "OEPS PN" ""
+		(property "OEPS PN" "OEPS010066"
 			(at 147.32 80.01 0)
 			(hide yes)
@@
 			)
 		)
-		(property "Description" "Resistor, US symbol"
+		(property "Description" "RESISTOR:   SMD 0805 0Ω 2A   [RC0805JR-070RL] [SMD]"
 			(at 121.92 92.71 0)
 			(hide yes)
@@
 			)
 		)
-		(property "MPN" ""
+		(property "MPN" "RC0805JR-070RL"
 			(at 121.92 92.71 90)
 			(hide yes)
@@
 			)
 		)
-		(property "OEPS PN" ""
+		(property "OEPS PN" "OEPS020025"
 			(at 121.92 92.71 90)
 			(hide yes)
@@
 			)
 		)
-		(property "Description" "Unpolarized capacitor"
+		(property "Description" "CAPACITOR:   SMD CER 0603 1uF 25V ±10% X5R   [CL10A105KA8NNNC] [SMD]"
 			(at 134.62 80.01 0)
 			(hide yes)
@@
 			)
 		)
-		(property "MPN" ""
+		(property "MPN" "CL10A105KA8NNNC"
 			(at 134.62 80.01 0)
 			(hide yes)
@@
 			)
 		)
-		(property "OEPS PN" ""
+		(property "OEPS PN" "OEPS010022"
 			(at 134.62 80.01 0)
 			(hide yes)
@@
 			)
 		)
-		(property "Description" "Resistor, US symbol"
+		(property "Description" "RESISTOR:   SMD 0805 0Ω 2A   [RC0805JR-070RL] [SMD]"
 			(at 121.92 107.95 0)
 			(hide yes)
@@
 			)
 		)
-		(property "MPN" ""
+		(property "MPN" "RC0805JR-070RL"
 			(at 121.92 107.95 90)
 			(hide yes)
@@
 			)
 		)
-		(property "OEPS PN" ""
+		(property "OEPS PN" "OEPS020025"
 			(at 121.92 107.95 90)
 			(hide yes)
@@
 			)
 		)
-		(property "Description" "Resistor, US symbol"
+		(property "Description" "RESISTOR:   SMD 0805 0Ω 2A   [RC0805JR-070RL] [SMD]"
 			(at 121.92 102.87 0)
 			(hide yes)
@@
 			)
 		)
-		(property "MPN" ""
+		(property "MPN" "RC0805JR-070RL"
 			(at 121.92 102.87 90)
 			(hide yes)
@@
 			)
 		)
-		(property "OEPS PN" ""
+		(property "OEPS PN" "OEPS020025"
 			(at 121.92 102.87 90)
 			(hide yes)
@@
 			)
 		)
-		(property "Description" "6-Channel Capacitive Touch Sensor, DFN-10"
+		(property "Description" "IC:   CAPACITIVE TOUCH SENSOR 6CH   [CAP1296-1-AIA-TR] [10-DFN-EP]"
 			(at 152.4 104.14 0)
 			(hide yes)
@@
 			)
 		)
-		(property "MPN" ""
+		(property "MPN" "CAP1296-1-AIA-TR"
 			(at 152.4 104.14 0)
 			(hide yes)
@@
 			)
 		)
-		(property "OEPS PN" ""
+		(property "OEPS PN" "OEPS080233"
 			(at 152.4 104.14 0)
 			(hide yes)
@@
 			)
 		)
-		(property "Description" "Resistor, US symbol"
+		(property "Description" "RESISTOR:   SMD 0805 0Ω 2A   [RC0805JR-070RL] [SMD]"
 			(at 121.92 97.79 0)
 			(hide yes)
@@
 			)
 		)
-		(property "MPN" ""
+		(property "MPN" "RC0805JR-070RL"
 			(at 121.92 97.79 90)
 			(hide yes)
@@
 			)
 		)
-		(property "OEPS PN" ""
+		(property "OEPS PN" "OEPS020025"
 			(at 121.92 97.79 90)
 			(hide yes)
