File: pcb/mcu-flash.kicad_sch (KiCad schematic)
At the start: 30 parts, among them J1 0015910100, SW1 EVQ-P7J01P, SW2 TS04-66-50-BK-160-SMT, U1 W25Q128JVS, U2 RP2040, Y1 ABM8AIG-12.000MHZ-12-2Z-T3

Commit message: Complete OEPS PN and manufacturing files
Parts:
- C1, C12: MPN (none) -> CL10A105KA8NNNC; OEPS PN (none) -> OEPS010022
- C10, C11, C13, C2, C3, C4, C5, C6, C7, C8, C9: MPN (none) -> C1005X5R1V104K050BB; OEPS PN (none) -> OEPS010066
- C14, C15: MPN (none) -> CL05C220JB51PNC; OEPS PN (none) -> OEPS010080
- J1: MPN (none) -> DNP; OEPS PN (none) -> OEPS000000
- R26, R27, R28, R29: MPN (none) -> RCS0402100RFKED; OEPS PN (none) -> OEPS020028
- R3, R5: MPN (none) -> RC0603FR-0710KL; OEPS PN (none) -> OEPS020133
- R4, R6: MPN (none) -> RMCF0402FT27R0; OEPS PN (none) -> OEPS020170
- R7: MPN (none) -> ERJ-2RKF1001X; OEPS PN (none) -> OEPS020006
- SW1: MPN (none) -> EVQ-P7J01P; OEPS PN (none) -> OEPS100090
- SW2: MPN (none) -> TS04-66-50-BK-160-SMT; OEPS PN (none) -> OEPS070115
- U1: MPN (none) -> W25Q128JVSIQ; OEPS PN (none) -> OEPS080163
- U2: MPN (none) -> SC0914(13); OEPS PN (none) -> OEPS080158
- Y1: MPN (none) -> ABM8AIG-12.000MHZ-12-2Z-T3; OEPS PN (none) -> OEPS100059
