File: pcb/oe-commutator-controller.kicad_sch (KiCad schematic)
At the start: 10 parts

Commit message: Exclude test points and capacitive touch from assembly position files
Also raised KiCAD version from 9 to 10.

These are non-assembly components that should not be included in pick-and-place machine files.

If possible, the Attributes for Test Points and Mounting Holes should be:
[X]  Exclude from bill of materials
[  ]  Exclude from board
[X]  Exclude from position files
[  ]  Do not populate
Parts:
- H1, H2, H3, H4, H5: value ~ -> (none)
- TP5, TP6: now left out of the parts list

Commit message: Complete OEPS PN and manufacturing files
Parts:
- R1, R2: MPN (none) -> RC0603FR-074K7L; OEPS PN (none) -> OEPS020236
- R30: MPN (none) -> RCS06030000Z0EA; OEPS PN (none) -> OEPS020151
Changed lines of the file:
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@@
 			)
 		)
-		(property "Description" "Resistor, US symbol"
+		(property "Description" "RESISTOR:   SMD 0603 4.7kΩ ±1% 0.100W   [RC0603FR-074K7L] [SMD]"
 			(at 101.6 68.58 0)
 			(hide yes)
@@
 			)
 		)
-		(property "MPN" ""
+		(property "MPN" "RC0603FR-074K7L"
 			(at 101.6 68.58 0)
 			(hide yes)
@@
 			)
 		)
-		(property "OEPS PN" ""
+		(property "OEPS PN" "OEPS020236"
 			(at 101.6 68.58 0)
 			(hide yes)
@@
 			)
 		)
-		(property "Description" "Resistor, US symbol"
+		(property "Description" "RESISTOR:   SMD 0603 0Ω 1A   [RCS06030000Z0EA] [SMD]"
 			(at 121.92 76.2 0)
 			(hide yes)
@@
 			)
 		)
-		(property "MPN" ""
+		(property "MPN" "RCS06030000Z0EA"
 			(at 121.92 76.2 90)
 			(hide yes)
@@
 			)
 		)
-		(property "OEPS PN" ""
+		(property "OEPS PN" "OEPS020151"
 			(at 121.92 76.2 90)
 			(hide yes)
@@
 			)
 		)
-		(property "Description" "Resistor, US symbol"
+		(property "Description" "RESISTOR:   SMD 0603 4.7kΩ ±1% 0.100W   [RC0603FR-074K7L] [SMD]"
 			(at 88.9 68.58 0)
 			(hide yes)
@@
 			)
 		)
-		(property "MPN" ""
+		(property "MPN" "RC0603FR-074K7L"
 			(at 88.9 68.58 0)
 			(hide yes)
@@
 			)
 		)
-		(property "OEPS PN" ""
+		(property "OEPS PN" "OEPS020236"
 			(at 88.9 68.58 0)
 			(hide yes)
