File: pcb/rgb-driver.kicad_sch (KiCad schematic)
At the start: 7 parts, among them U8 IS31FL3193

Commit message: Complete OEPS PN and manufacturing files
Parts:
- C35, C37: MPN (none) -> GRM21BR61H475KE51L; OEPS PN (none) -> OEPS010013
- C36: MPN (none) -> CGA2B3X7R1H104K050BB; OEPS PN (none) -> OEPS010016
- D1: MPN (none) -> XZMDKCBDDG45S-9; OEPS PN (none) -> OEPS030057
- R23, R24: MPN (none) -> RC0603FR-0710KL; OEPS PN (none) -> OEPS020133
- U8: MPN (none) -> IS31FL3193-DLS2-TR; OEPS PN (none) -> OEPS080232
Changed lines of the file:
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@@
 			)
 		)
-		(property "Description" "Unpolarized capacitor"
+		(property "Description" "CAPACITOR:   SMD CER 0805 4.7uF 50V ±10% X5R   [GRM21BR61H475KE51L] [SMD]"
 			(at 69.85 76.2 0)
 			(hide yes)
@@
 			)
 		)
-		(property "MPN" ""
+		(property "MPN" "GRM21BR61H475KE51L"
 			(at 69.85 76.2 0)
 			(hide yes)
@@
 			)
 		)
-		(property "OEPS PN" ""
+		(property "OEPS PN" "OEPS010013"
 			(at 69.85 76.2 0)
 			(hide yes)
@@
 			)
 		)
-		(property "Description" "Resistor, US symbol"
+		(property "Description" "RESISTOR:   SMD 0603 10kΩ ±1% 0.100W   [RC0603FR-0710KL] [SMD]"
 			(at 156.21 93.98 0)
 			(hide yes)
@@
 			)
 		)
-		(property "MPN" ""
+		(property "MPN" "RC0603FR-0710KL"
 			(at 156.21 93.98 0)
 			(hide yes)
@@
 			)
 		)
-		(property "OEPS PN" ""
+		(property "OEPS PN" "OEPS020133"
 			(at 156.21 93.98 0)
 			(hide yes)
@@
 			)
 		)
-		(property "Description" "Unpolarized capacitor"
+		(property "Description" "CAPACITOR:   SMD CER 0402 100nF 50V ±10% X7R   [CGA2B3X7R1H104K050BB] [SMD]"
 			(at 175.26 92.71 0)
 			(hide yes)
@@
 			)
 		)
-		(property "MPN" ""
+		(property "MPN" "CGA2B3X7R1H104K050BB"
 			(at 175.26 92.71 0)
 			(hide yes)
@@
 			)
 		)
-		(property "OEPS PN" ""
+		(property "OEPS PN" "OEPS010016"
 			(at 175.26 92.71 0)
 			(hide yes)
@@
 			)
 		)
-		(property "Description" "Unpolarized capacitor"
+		(property "Description" "CAPACITOR:   SMD CER 0805 4.7uF 50V ±10% X5R   [GRM21BR61H475KE51L] [SMD]"
 			(at 185.42 101.6 0)
 			(hide yes)
@@
 			)
 		)
-		(property "MPN" ""
+		(property "MPN" "GRM21BR61H475KE51L"
 			(at 185.42 101.6 0)
 			(hide yes)
@@
 			)
 		)
-		(property "OEPS PN" ""
+		(property "OEPS PN" "OEPS010013"
 			(at 185.42 101.6 0)
 			(hide yes)
@@
 			)
 		)
-		(property "Description" "Resistor, US symbol"
+		(property "Description" "RESISTOR:   SMD 0603 10kΩ ±1% 0.100W   [RC0603FR-0710KL] [SMD]"
 			(at 156.21 113.03 0)
 			(hide yes)
@@
 			)
 		)
-		(property "MPN" ""
+		(property "MPN" "RC0603FR-0710KL"
 			(at 156.21 113.03 0)
 			(hide yes)
@@
 			)
 		)
-		(property "OEPS PN" ""
+		(property "OEPS PN" "OEPS020133"
 			(at 156.21 113.03 0)
 			(hide yes)
@@
 			)
 		)
-		(property "Description" "RGB LED, red/anode/blue/green"
+		(property "Description" "DIODE:   LED SMD RGB Red 645nm Green 515nm Blue 460nm   [XZMDKCBDDG45S-9] [4-PLCC]"
 			(at 87.63 82.55 0)
 			(hide yes)
@@
 			)
 		)
-		(property "MPN" ""
+		(property "MPN" "XZMDKCBDDG45S-9"
 			(at 87.63 82.55 90)
 			(hide yes)
@@
 			)
 		)
-		(property "OEPS PN" ""
+		(property "OEPS PN" "OEPS030057"
 			(at 87.63 82.55 90)
 			(hide yes)
@@
 			)
 		)
-		(property "Description" "3-CHANNEL LED DRIVER"
+		(property "Description" "IC:   LED DRIVER LINEAR 42MA   [IS31FL3193-DLS2-TR] [10-DFN-EP]"
 			(at 130.81 100.33 0)
 			(hide yes)
@@
 			)
 		)
-		(property "MPN" ""
+		(property "MPN" "IS31FL3193-DLS2-TR"
 			(at 130.81 100.33 0)
 			(hide yes)
@@
 			)
 		)
-		(property "OEPS PN" ""
+		(property "OEPS PN" "OEPS080232"
 			(at 130.81 100.33 0)
 			(hide yes)
