File: pcb/usb-power.kicad_sch (KiCad schematic)
At the start: 10 parts, among them J2 USB4110-GF-A, U9 AP2112K-3.3

Commit message: Exclude test points and capacitive touch from assembly position files
Also raised KiCAD version from 9 to 10.

These are non-assembly components that should not be included in pick-and-place machine files.

If possible, the Attributes for Test Points and Mounting Holes should be:
[X]  Exclude from bill of materials
[  ]  Exclude from board
[X]  Exclude from position files
[  ]  Do not populate
Parts:
- TP1, TP4: value ~ -> (none)

Commit message: Complete OEPS PN and manufacturing files
Parts:
- C18: MPN (none) -> C1005X5R1V104K050BB; OEPS PN (none) -> OEPS010066
- C38, C39: MPN (none) -> CL10A105KA8NNNC; OEPS PN (none) -> OEPS010022
- D9: MPN (none) -> TPD4E05U06DQAR; OEPS PN (none) -> OEPS030037
- J2: MPN (none) -> USB4110-GF-A; OEPS PN (none) -> OEPS070153
- R8, R9: MPN (none) -> ERJ-2RKF5101X; OEPS PN (none) -> OEPS020173
- TP1, TP4: now left out of the parts list
- U9: MPN (none) -> AP2112K-3.3TRG1; OEPS PN (none) -> OEPS080155
Changed lines of the file:
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@@
 		(body_style 1)
 		(exclude_from_sim no)
-		(in_bom yes)
-		(on_board yes)
-		(in_pos_files yes)
+		(in_bom no)
+		(on_board yes)
+		(in_pos_files no)
 		(dnp no)
 		(property "Reference" "TP4"
@@
 			)
 		)
-		(property "Description" "test point"
+		(property "Description" "#N/A"
 			(at 204.47 102.87 0)
 			(hide yes)
@@
 			)
 		)
-		(property "Description" "Unpolarized capacitor, small symbol"
+		(property "Description" "CAPACITOR:   SMD CER 0402 100nF 35V ±10% X5R (OEPS H1 001)   [C1005X5R1V104K050BB] [SMD]"
 			(at 124.46 113.03 0)
 			(hide yes)
@@
 			)
 		)
-		(property "MPN" ""
+		(property "MPN" "C1005X5R1V104K050BB"
 			(at 124.46 113.03 0)
 			(hide yes)
@@
 			)
 		)
-		(property "OEPS PN" ""
+		(property "OEPS PN" "OEPS010066"
 			(at 124.46 113.03 0)
 			(hide yes)
@@
 			)
 		)
-		(property "Description" "Resistor, US symbol"
+		(property "Description" "RESISTOR:   SMD 0402 5.1kΩ ±1% 0.100W   [ERJ-2RKF5101X] [SMD]"
 			(at 143.51 110.49 0)
 			(hide yes)
@@
 			)
 		)
-		(property "MPN" ""
+		(property "MPN" "ERJ-2RKF5101X"
 			(at 143.51 110.49 90)
 			(hide yes)
@@
 			)
 		)
-		(property "OEPS PN" ""
+		(property "OEPS PN" "OEPS020173"
 			(at 143.51 110.49 90)
 			(hide yes)
@@
 			)
 		)
-		(property "Description" "600mA low dropout linear regulator, with enable pin, 3.8V-6V input voltage range, 3.3V fixed positive output, SOT-23-5"
+		(property "Description" "IC:   LDO 3.3V 600mA   [AP2112K-3.3TRG1] [SOT-23-5]"
 			(at 194.31 106.68 0)
 			(hide yes)
@@
 			)
 		)
-		(property "MPN" ""
+		(property "MPN" "AP2112K-3.3TRG1"
 			(at 194.31 106.68 0)
 			(hide yes)
@@
 			)
 		)
-		(property "OEPS PN" ""
+		(property "OEPS PN" "OEPS080155"
 			(at 194.31 106.68 0)
 			(hide yes)
@@
 			)
 		)
-		(property "Description" "USB 2.0-only 16P Type-C Receptacle connector"
+		(property "Description" "CONNECTOR:   USB2.0 TYPE C 24P SMD R/A   [USB4110-GF-A] [SMD]"
 			(at 106.68 88.9 0)
 			(hide yes)
@@
 			)
 		)
-		(property "MPN" ""
+		(property "MPN" "USB4110-GF-A"
 			(at 106.68 88.9 0)
 			(hide yes)
@@
 			)
 		)
-		(property "OEPS PN" ""
+		(property "OEPS PN" "OEPS070153"
 			(at 106.68 88.9 0)
 			(hide yes)
@@
 			)
 		)
-		(property "Description" "Resistor, US symbol"
+		(property "Description" "RESISTOR:   SMD 0402 5.1kΩ ±1% 0.100W   [ERJ-2RKF5101X] [SMD]"
 			(at 138.43 110.49 0)
 			(hide yes)
@@
 			)
 		)
-		(property "MPN" ""
+		(property "MPN" "ERJ-2RKF5101X"
 			(at 138.43 110.49 90)
 			(hide yes)
@@
 			)
 		)
-		(property "OEPS PN" ""
+		(property "OEPS PN" "OEPS020173"
 			(at 138.43 110.49 90)
 			(hide yes)
@@
 			)
 		)
-		(property "Description" "4-Channel ESD Protection for Super-Speed USB 3.0 Interface, USON-10"
+		(property "Description" "DIODE:   TVS DIODE 5.5VWM 14VC   [TPD4E05U06DQAR] [10-UFDFN]"
 			(at 194.31 73.66 0)
 			(hide yes)
@@
 			)
 		)
-		(property "MPN" ""
+		(property "MPN" "TPD4E05U06DQAR"
 			(at 194.31 73.66 0)
 			(hide yes)
@@
 			)
 		)
-		(property "OEPS PN" ""
+		(property "OEPS PN" "OEPS030037"
 			(at 194.31 73.66 0)
 			(hide yes)
@@
 		(body_style 1)
 		(exclude_from_sim no)
-		(in_bom yes)
-		(on_board yes)
-		(in_pos_files yes)
+		(in_bom no)
+		(on_board yes)
+		(in_pos_files no)
 		(dnp no)
 		(property "Reference" "TP1"
@@
 			)
 		)
-		(property "Description" "test point"
+		(property "Description" "#N/A"
 			(at 165.1 104.14 0)
 			(hide yes)
@@
 			)
 		)
-		(property "Description" "Unpolarized capacitor"
+		(property "Description" "CAPACITOR:   SMD CER 0603 1uF 25V ±10% X5R   [CL10A105KA8NNNC] [SMD]"
 			(at 173.99 110.49 0)
 			(hide yes)
@@
 			)
 		)
-		(property "MPN" ""
+		(property "MPN" "CL10A105KA8NNNC"
 			(at 173.99 110.49 0)
 			(hide yes)
@@
 			)
 		)
-		(property "OEPS PN" ""
+		(property "OEPS PN" "OEPS010022"
 			(at 173.99 110.49 0)
 			(hide yes)
@@
 			)
 		)
-		(property "Description" "Unpolarized capacitor"
+		(property "Description" "CAPACITOR:   SMD CER 0603 1uF 25V ±10% X5R   [CL10A105KA8NNNC] [SMD]"
 			(at 210.82 110.49 0)
 			(hide yes)
@@
 			)
 		)
-		(property "MPN" ""
+		(property "MPN" "CL10A105KA8NNNC"
 			(at 210.82 110.49 0)
 			(hide yes)
@@
 			)
 		)
-		(property "OEPS PN" ""
+		(property "OEPS PN" "OEPS010022"
 			(at 210.82 110.49 0)
 			(hide yes)
